Commit message: shoulder and shoulder arm and joint done in urdf (J2)

File: src/bin_nodes/urdf/robot.urdf (robot description, URDF)
Before this commit: robot robot_arm, 2 links, 1 joints
Links:
- added link shoulder_arm; collision cylinder length=0.3 radius=0.04; visual cylinder length=0.3 radius=0.04
- added link shoulder_link; collision cylinder length=0.14 radius=0.04; visual cylinder length=0.14 radius=0.04
Joints:
- added joint a1_shoulder: type fixed, parent shoulder_link, child shoulder_arm, origin xyz=0.02 0 0.15 rpy=0 0 0
- added joint j2_shoulder: type revolute, parent waist_link, child shoulder_link, origin xyz=0.10 0 0.02 rpy=0 0 0, axis 1 0 0, limit lower=-3.14159 upper=3.14159 effort=100.0 velocity=1.0

File: src/install/bin_nodes/share/bin_nodes/urdf/robot.urdf (robot description, URDF)
Before this commit: robot robot_arm, 2 links, 1 joints
Links:
- added link shoulder_arm; collision cylinder length=0.3 radius=0.04; visual cylinder length=0.3 radius=0.04
- added link shoulder_link; collision cylinder length=0.14 radius=0.04; visual cylinder length=0.14 radius=0.04
Joints:
- added joint a1_shoulder: type fixed, parent shoulder_link, child shoulder_arm, origin xyz=0.02 0 0.15 rpy=0 0 0
- added joint j2_shoulder: type revolute, parent waist_link, child shoulder_link, origin xyz=0.10 0 0.02 rpy=0 0 0, axis 1 0 0, limit lower=-3.14159 upper=3.14159 effort=100.0 velocity=1.0

Commit message: finished elbow elbow arm and joint (J3)

File: src/bin_nodes/urdf/robot.urdf (robot description, URDF)
Before this commit: robot robot_arm, 4 links, 3 joints
Links:
- added link elbow_arm; collision cylinder length=0.35 radius=0.04; visual cylinder length=0.35 radius=0.04
- added link elbow_link; collision cylinder length=0.16 radius=0.04; visual cylinder length=0.16 radius=0.04
- link shoulder_arm: geometry collision cylinder length=0.35 radius=0.04; visual cylinder length=0.35 radius=0.04
Joints:
- added joint a2_elbow: type fixed, parent elbow_link, child elbow_arm, origin xyz=-0.04 0 0.18 rpy=0 0 0
- added joint j3_elbow: type revolute, parent shoulder_arm, child elbow_link, origin xyz=-0.09 0 0.134 rpy=0 0 0, axis 1 0 0, limit lower=-3.14159 upper=3.14159 effort=100.0 velocity=1.0
- joint a1_shoulder: origin xyz=0.02 0 0.15 rpy=0 0 0 -> xyz=0.027 0 0.18 rpy=0 0 0

File: src/install/bin_nodes/share/bin_nodes/urdf/robot.urdf (robot description, URDF)
Before this commit: robot robot_arm, 4 links, 3 joints
Links:
- added link elbow_arm; collision cylinder length=0.35 radius=0.04; visual cylinder length=0.35 radius=0.04
- added link elbow_link; collision cylinder length=0.16 radius=0.04; visual cylinder length=0.16 radius=0.04
- link shoulder_arm: geometry collision cylinder length=0.35 radius=0.04; visual cylinder length=0.35 radius=0.04
Joints:
- added joint a2_elbow: type fixed, parent elbow_link, child elbow_arm, origin xyz=-0.04 0 0.18 rpy=0 0 0
- added joint j3_elbow: type revolute, parent shoulder_arm, child elbow_link, origin xyz=-0.09 0 0.134 rpy=0 0 0, axis 1 0 0, limit lower=-3.14159 upper=3.14159 effort=100.0 velocity=1.0
- joint a1_shoulder: origin xyz=0.02 0 0.15 rpy=0 0 0 -> xyz=0.027 0 0.18 rpy=0 0 0

Commit message: finished wrist roll (J4)

File: src/bin_nodes/urdf/robot.urdf (robot description, URDF)
Before this commit: robot robot_arm, 6 links, 5 joints
Links:
- added link wrist_link; collision cylinder length=0.03 radius=0.04; visual cylinder length=0.03 radius=0.04
Joints:
- added joint j4_wrist: type revolute, parent elbow_arm, child wrist_link, origin xyz=0 0 0.19 rpy=0 0 0, axis 0 0 1, limit lower=-3.14159 upper=3.14159 effort=100.0 velocity=1.0

Commit message: finished wrist pitch (J5)

File: src/bin_nodes/urdf/robot.urdf (robot description, URDF)
Before this commit: robot robot_arm, 7 links, 6 joints
Links:
- added link wrist_arm; collision cylinder length=0.08 radius=0.02; visual cylinder length=0.08 radius=0.02
- added link wrist_pitch_link; collision cylinder length=0.08 radius=0.02; visual cylinder length=0.08 radius=0.02
- added link wrist_yaw_link; collision sphere radius=0.03; visual sphere radius=0.03
- link wrist_link: geometry collision cylinder length=0.05 radius=0.04; visual cylinder length=0.05 radius=0.04
Joints:
- added joint a3_wrist: type fixed, parent wrist_pitch_link, child wrist_arm, origin xyz=0.01 0 0.04 rpy=0 0 0
- added joint j5_wrist: type revolute, parent wrist_link, child wrist_pitch_link, origin xyz=0.06 0 0 rpy=0 0 0, axis 1 0 0, limit lower=-3.14159 upper=3.14159 effort=100.0 velocity=1.0
- added joint j6_wrist: type revolute, parent wrist_arm, child wrist_yaw_link, origin xyz=0 0 0.05 rpy=0 0 0, axis 0 1 0, limit lower=-3.14159 upper=3.14159 effort=100.0 velocity=1.0
- joint j4_wrist: origin xyz=0 0 0.19 rpy=0 0 0 -> xyz=0 0 0.2 rpy=0 0 0

Commit message: finished wrist yaw (J6) and added mock tool

File: src/bin_nodes/urdf/robot.urdf (robot description, URDF)
Before this commit: robot robot_arm, 10 links, 9 joints
Links:
- added link tool_link; collision cylinder length=0.05 radius=0.01; visual cylinder length=0.05 radius=0.01
- link wrist_yaw_link: geometry collision sphere radius=0.02; visual sphere radius=0.02
Joints:
- added joint tool_joint: type fixed, parent wrist_yaw_link, child tool_link, origin xyz=0 0 0.04 rpy=0 0 0
- joint a3_wrist: origin xyz=0.01 0 0.04 rpy=0 0 0 -> xyz=0.02 0 0.04 rpy=0 0 0
- joint j6_wrist: limit lower=-3.14159 upper=3.14159 effort=100.0 velocity=1.0 -> lower=-1.54159 upper=1.54159 effort=100.0 velocity=1.0; origin xyz=0 0 0.05 rpy=0 0 0 -> xyz=0 0 0.04 rpy=0 0 0
