Commit message: edited the collision boxes in urdf for better movement

File: install/bin_nodes/share/bin_nodes/urdf/robot.urdf (robot description, URDF)
Before this commit: robot robot_arm, 11 links, 10 joints
Links:
- link elbow_arm: geometry collision cylinder length=0.35 radius=0.04; visual cylinder length=0.35 radius=0.04
- link elbow_link: geometry collision cylinder length=0.16 radius=0.04; visual cylinder length=0.16 radius=0.04
- link robot_base: geometry collision box size=0.2 0.2 0.05; visual box size=0.2 0.2 0.05
- link shoulder_arm: geometry collision cylinder length=0.35 radius=0.04; visual cylinder length=0.35 radius=0.04
- link shoulder_link: geometry collision cylinder length=0.14 radius=0.04; visual cylinder length=0.14 radius=0.04
- link tool_link: geometry collision cylinder length=0.05 radius=0.01; visual cylinder length=0.05 radius=0.01
- link waist_link: geometry collision cylinder length=0.15 radius=0.06; visual cylinder length=0.15 radius=0.06
- link wrist_arm: geometry collision cylinder length=0.08 radius=0.02; visual cylinder length=0.08 radius=0.02
- link wrist_link: geometry collision cylinder length=0.05 radius=0.04; visual cylinder length=0.05 radius=0.04
- link wrist_pitch_link: geometry collision cylinder length=0.08 radius=0.02; visual cylinder length=0.08 radius=0.02
- link wrist_yaw_link: geometry collision sphere radius=0.02; visual sphere radius=0.02

Commit message: moveit setup done

File: install/bin_nodes/share/bin_nodes/urdf/robot.urdf (robot description, URDF)
Before this commit: robot robot_arm, 11 links, 10 joints
Links:
- link elbow_arm: geometry collision box size=0.06 0.06 0.31; visual cylinder length=0.35 radius=0.04
- link elbow_link: geometry collision box size=0.06 0.06 0.14; visual cylinder length=0.16 radius=0.04
- link robot_base: geometry collision box size=0.18 0.18 0.04; visual box size=0.2 0.2 0.05
- link shoulder_arm: geometry collision box size=0.06 0.06 0.31; visual cylinder length=0.35 radius=0.04
- link shoulder_link: geometry collision box size=0.06 0.06 0.12; visual cylinder length=0.14 radius=0.04
- link tool_link: geometry collision box size=0.015 0.015 0.04; visual cylinder length=0.05 radius=0.01
- link waist_link: geometry collision box size=0.09 0.09 0.13; visual cylinder length=0.15 radius=0.06
- link wrist_arm: geometry collision box size=0.03 0.03 0.05; visual cylinder length=0.08 radius=0.02
- link wrist_link: geometry collision box size=0.06 0.06 0.04; visual cylinder length=0.05 radius=0.04
- link wrist_pitch_link: geometry collision box size=0.03 0.03 0.04; visual cylinder length=0.08 radius=0.02
- link wrist_yaw_link: geometry collision sphere radius=0.015; visual sphere radius=0.02

Commit message: added gripper to urdf

File: install/bin_nodes/share/bin_nodes/urdf/robot.urdf (robot description, URDF)
Before this commit: robot robot_arm, 11 links, 10 joints
Links:
- added link gripper_link; collision box size=0.015 0.015 0.03; visual box size=0.015 0.015 0.05
- added link gripperfinger_left_link; collision box size=0.0075 0.0075 0.04; visual box size=0.0075 0.0075 0.04
- added link gripperfinger_right_link; collision box size=0.0075 0.0075 0.04; visual box size=0.0075 0.0075 0.04
- link tool_link: geometry collision box size=0.015 0.015 0.03; visual cylinder length=0.04 radius=0.01
Joints:
- added joint gripper_joint: type fixed, parent tool_link, child gripper_link, origin xyz=0 0 0.02 rpy=0 0 0
- added joint gripperfinger_left_joint: type prismatic, parent gripper_link, child gripperfinger_left_link, origin xyz=0 0.02 0.02 rpy=0 0 0, axis 0 -1 0, limit lower=0 upper=0.02 effort=100.0 velocity=1.0
- added joint gripperfinger_right_joint: type prismatic, parent gripper_link, child gripperfinger_right_link, origin xyz=0 -0.02 0.02 rpy=0 0 0, axis 0 1 0, limit lower=0 upper=0.02 effort=100.0 velocity=1.0
- joint tool_joint: origin xyz=0 0 0.04 rpy=0 0 0 -> xyz=0 0 0.03 rpy=0 0 0
