Commit message: finally got the moveit control to work directly with gazebo

File: install/bin_nodes/share/bin_nodes/urdf/robot.urdf (robot description, URDF)
Before this commit: robot robot_arm, 14 links, 13 joints
Links:
- link elbow_arm: mass None -> 0.8
- link elbow_link: mass None -> 0.5
- link gripper_link: mass None -> 0.05
- link gripperfinger_left_link: mass None -> 0.02
- link gripperfinger_right_link: mass None -> 0.02
- link robot_base: mass None -> 2.0
- link shoulder_arm: mass None -> 0.8
- link shoulder_link: mass None -> 0.5
- link tool_link: mass None -> 0.05
- link waist_link: mass None -> 1.0
- link wrist_arm: mass None -> 0.2
- link wrist_link: mass None -> 0.3
- link wrist_pitch_link: mass None -> 0.2
- link wrist_yaw_link: mass None -> 0.1

File: install/moveit_config/share/moveit_config/config/robot_arm.ros2_control.xacro (robot description, xacro)
@@ -1,10 +1,16 @@
 <?xml version="1.0"?>
 <robot xmlns:xacro="http://www.ros.org/wiki/xacro">
-    <xacro:macro name="robot_arm_ros2_control" params="name initial_positions_file">
+    <xacro:macro name="robot_arm_ros2_control" params="name initial_positions_file use_gazebo:=false">
         <xacro:property name="initial_positions" value="${load_yaml(initial_positions_file)['initial_positions']}"/>
         <ros2_control name="${name}" type="system">
             <hardware>
-                <!-- By default, set up controllers for simulation. This won't work on real hardware -->
-                <plugin>mock_components/GenericSystem</plugin>
+                <xacro:if value="${use_gazebo}">
+                    <!-- Gazebo Classic: the controller_manager runs inside Gazebo -->
+                    <plugin>gazebo_ros2_control/GazeboSystem</plugin>
+                </xacro:if>
+                <xacro:unless value="${use_gazebo}">
+                    <!-- Mock hardware for the RViz-only demo (no physics) -->
+                    <plugin>mock_components/GenericSystem</plugin>
+                </xacro:unless>
             </hardware>
             <joint name="j1_waist">

File: install/moveit_config/share/moveit_config/config/robot_arm.urdf.xacro (robot description, xacro)
@@ -2,8 +2,23 @@
 <robot xmlns:xacro="http://www.ros.org/wiki/xacro" name="robot_arm">
     <xacro:arg name="initial_positions_file" default="initial_positions.yaml" />
+    <!-- Set to true when launching in Gazebo (see gazebo.launch.py). Leave false for the RViz demo. -->
+    <xacro:arg name="use_gazebo" default="false" />
     <!-- Import robot_arm urdf file -->
     <xacro:include filename="$(find bin_nodes)/urdf/robot.urdf" />
     <!-- Import control_xacro -->
     <xacro:include filename="robot_arm.ros2_control.xacro" />
-    <xacro:robot_arm_ros2_control name="FakeSystem" initial_positions_file="$(arg initial_positions_file)"/>
+    <xacro:robot_arm_ros2_control name="FakeSystem" initial_positions_file="$(arg initial_positions_file)" use_gazebo="$(arg use_gazebo)"/>
+    <!-- Gazebo-only: anchor the base to the world frame and load the ros2_control plugin. -->
+    <xacro:if value="$(arg use_gazebo)">
+        <link name="world"/>
+        <joint name="world_fixed" type="fixed">
+            <parent link="world"/>
+            <child link="robot_base"/>
+        </joint>
+        <gazebo>
+            <plugin filename="libgazebo_ros2_control.so" name="gazebo_ros2_control">
+                <parameters>$(find moveit_config)/config/ros2_controllers.yaml</parameters>
+            </plugin>
+        </gazebo>
+    </xacro:if>
 </robot>
