Commit message: added new VisionNode and now it takes the depth image and displays it

File: install/bin_nodes/share/bin_nodes/urdf/camera.urdf (robot description, URDF)
Before this commit: robot camera, 3 links, 2 joints
Joints:
- joint camera_mount_joint: origin xyz=0.4 0 1.4 rpy=0 1.5708 0 -> xyz=0.4 0.35 1.1 rpy=0 1.5708 0
