Commit message: edited the moveit config to include the gripper planning group and the new end effector group

File: install/moveit_config/share/moveit_config/config/robot_arm.ros2_control.xacro (robot description, xacro)
@@ -44,4 +44,16 @@
                 </state_interface>
             </joint>
+            <joint name="gripperfinger_left_joint">
+                <command_interface name="position"/>
+                <state_interface name="position">
+                  <param name="initial_value">${initial_positions['gripperfinger_left_joint']}</param>
+                </state_interface>
+            </joint>
+            <joint name="gripperfinger_right_joint">
+                <command_interface name="position"/>
+                <state_interface name="position">
+                  <param name="initial_value">${initial_positions['gripperfinger_right_joint']}</param>
+                </state_interface>
+            </joint>
         </ros2_control>
     </xacro:macro>
